File: PCB/Auth75.kicad_sch (KiCad schematic)
At the start: 193 parts, among them Q1 MMBT3904LT1G, Q2 MMBT3904LT1G, Q3 MMBT3904LT1G, Q4 MMBT3906LT1G, SW1 EC11E15244G1, U1 RASPBERRY PI PICO 2W, U2 SL2.1S

Commit message: adding battery charger
Parts:
- added C13, C9: 4.7uF, Capacitor_SMD:C_0603_1608Metric, symbol Device:C
- added C14: 100nF, Capacitor_SMD:C_0603_1608Metric, symbol Device:C
- added CN1: S2B-PH-SM4-TB, easyeda2kicad:CONN-SMD_P2.00_S2B-PH-SM4-TB-LF-SN, symbol easyeda2kicad:S2B-PH-SM4-TB
- added D81: LED, LED_SMD:LED_0603_1608Metric, symbol Device:LED
- added D82: (no value), Diode_SMD:D_SOD-123, symbol ScottoKeebs:Placeholder_Diode
- added Q5: FS8205A_C2830320, easyeda2kicad:SOT-23-6_L2.9-W1.6-P0.95-LS2.8-BR, symbol easyeda2kicad:FS8205A_C2830320
- added R13: 470, Resistor_SMD:R_0603_1608Metric, symbol Device:R
- added R14: 2k, Resistor_SMD:R_0603_1608Metric, symbol Device:R
- added R15: 100, Resistor_SMD:R_0603_1608Metric, symbol Device:R
- added R16: 1k, Resistor_SMD:R_0603_1608Metric, symbol Device:R
- added R17, R18: 4.7k, Resistor_SMD:R_0603_1608Metric, symbol Device:R
- added U3: DW01A_C351410, easyeda2kicad:SOT-23-6_L2.9-W1.6-P0.95-LS2.8-BL, symbol easyeda2kicad:DW01A_C351410
- added U4: MCP73831T-2ACI/OT, easyeda2kicad:SOT-23-5_L3.0-W1.7-P0.95-LS2.8-BL, symbol easyeda2kicad:MCP73831T-2ACI_OT
- added U5: PCA9536DGKR, easyeda2kicad:VSSOP-8_L3.0-W3.0-P0.65-LS4.9-BL, symbol easyeda2kicad:PCA9536DGKR
- C1, C10, C11, C12, C2, C3, C5, C7: LCSC Part (none) -> C15849
- C4, C6, C8: LCSC Part (none) -> C14663
- D1, D10, D11, D12, D13, D14, D15, D16, D17, D18, D19, D2, D20, D21, D22, D23, D24, D25, D26, D27, D28, D29, D3, D30, D31, D32, D33, D34, D35, D36, D37, D38, D39, D4, D40, D41, D42, D43, D44, D45, D46, D47, D48, D49, D5, D50, D51, D52, D53, D54, D55, D56, D57, D58, D59, D6, D60, D61, D62, D63, D64, D65, D66, D67, D68, D69, D7, D70, D71, D72, D73, D74, D75, D76, D77, D78, D79, D8, D80, D9: LCSC Part (none) -> C81598
- R1, R2, R3, R4, R5, R6, R7, R8: LCSC Part (none) -> C23186
- R10, R11, R9: LCSC Part (none) -> C21190
- R12: LCSC Part (none) -> C25804
- S1, S10, S11, S12, S13, S14, S15, S16, S17, S18, S19, S2, S20, S21, S22, S23, S24, S25, S26, S27, S28, S29, S3, S30, S31, S32, S33, S34, S35, S36, S37, S38, S39, S4, S40, S41, S42, S43, S44, S45, S46, S47, S48, S49, S5, S50, S51, S52, S53, S54, S55, S56, S57, S58, S59, S6, S60, S61, S62, S63, S64, S65, S66, S67, S68, S69, S7, S70, S71, S72, S73, S74, S75, S76, S77, S78, S8, S9: LCSC Part (none) -> C2803348
- SW1: now left out of the parts list
Connections:
- net +3.3V: now also R17.2, R18.2, U5.8 (VCC)
- net +5V: now also C9.1, D81.2 (A), U4.4 (VDD)
- net Fprint LED Green MCU: now also U5.2 (P1); no longer U1.31 (GP26_ADC0_I2C1SDA)
- net Fprint LED Red MCU: now also U5.3 (P2); no longer U1.32 (GP27_ADC1_I2C1SCL)
- net Fprint LED White MCU: now also U5.1 (P0); no longer U1.29 (GP22)
- net Fprint Touch: now also U5.5 (P3); no longer U1.34 (GP28_ADC2)
- net GND: now also C13.2, C9.2, CN1.3, CN1.4, Q5.3 (S2), R14.1, U4.2 (VSS), U5.4 (GND)
- net at U1.39 (VSYS): now also D82.1 (K)
- new net: D81.1 (K), R13.1
- new net: Q5.6 (G1), U3.1 (OD)
- new net: R16.2, U3.2 (VM)
- new net: Q5.4 (G2), U3.3 (OC)
- new net: C14.2, R15.1, U3.5 (VCC)
- new net: R14.2, U4.5 (PROG)
- new net BATT+: C13.1, CN1.1, D82.2 (A), R15.2, U4.3 (VBAT)
- new net BATT-: C14.1, CN1.2, Q5.1 (S1), U3.6 (GND)
- new net D1/D2: Q5.2 (D1/D2), Q5.5 (D1/D2), R16.1
- new net PCA9536DGKR SCL: R18.1, U1.32 (GP27_ADC1_I2C1SCL), U5.6 (SCL)
- new net PCA9536DGKR SDA: R17.1, U1.31 (GP26_ADC0_I2C1SDA), U5.7 (SDA)
- new net STAT: R13.2, U1.29 (GP22), U4.1 (STAT)
- no-connect marks 15 -> 16
