File: PCB/Auth75.kicad_sch (KiCad schematic)
At the start: 209 parts, among them CN1 S2B-PH-SM4-TB, Q1 MMBT3904LT1G, Q2 MMBT3904LT1G, Q3 MMBT3904LT1G, Q4 MMBT3906LT1G, Q5 FS8205A_C2830320, SW1 EC11E15244G1, U1 RASPBERRY PI PICO 2W, U2 SL2.1S, U3 DW01A_C351410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

Commit message: Wrap up project and adding silkscreen
Parts:
- R14: LCSC Part C4180 -> C22975
- R15: LCSC Part C25076 -> C22775
Changed lines of the file:
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@@
 			)
 		)
-		(property "LCSC Part" "C25076"
+		(property "LCSC Part" "C22775"
 			(at 266.7 82.55 90)
 			(hide yes)
@@
 			)
 		)
-		(property "LCSC Part" "C4180"
+		(property "LCSC Part" "C22975"
 			(at 254 27.94 0)
 			(hide yes)
