File: PCB_Cheap/Auth75.kicad_pcb (KiCad board)
At the start: 2 copper layers, 326.7 x 132.3 mm, 232 parts, among them CN1 S2B-PH-SM4-TB, Q1 MMBT3904-C20526, Q2 MMBT3904-C20526, Q3 MMBT3904-C20526, Q4 SS8550_C8542, Q5 FS8205A_C2830320, SW1 EC11E15244G1, U1 RASPBERRY PI PICO 2W, U2 SL2.1S, U3 DW01A_C351410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

Commit message: 56k resis for pull up
Parts:
- R3, R4, R5, R6, R7, R8: value 5.1k -> 56k
